File: piano-keyboard-end-pcb/piano-keyboard-end-pcb.sch (KiCad schematic (older format))
At the start: 21 parts, among them J1 Conn_01x03_Male, J2 Conn_01x01_Male, J3 Conn_01x02_Male, J4 Conn_01x02_Male, J5 Conn_01x05_Female, J6 AudioJack2, SW1 SW_Push, SW2 SW_Push, SW3 SW_Push, SW4 SW_Push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

Commit message: start laying out end pcb
Parts:
- J1: footprint (none) -> Connector_PinHeader_2.54mm:PinHeader_1x03_P2.54mm_Vertical
- J2: footprint (none) -> Connector_PinHeader_2.54mm:PinHeader_1x01_P2.54mm_Vertical
- J3, J4: footprint (none) -> Connector_PinHeader_2.54mm:PinHeader_1x02_P2.54mm_Vertical
- R1, R2, R3: footprint (none) -> Resistor_THT:R_Axial_DIN0207_L6.3mm_D2.5mm_P7.62mm_Horizontal
Changed lines of the file:
@@
 EESchema Schematic File Version 4
+LIBS:piano-keyboard-end-pcb-cache
 EELAYER 29 0
 EELAYER END
@@
 F 0 "J1" H 2908 2931 50  0000 C CNN
 F 1 "Conn_01x03_Male" H 2908 2840 50  0000 C CNN
-F 2 "" H 2800 2650 50  0001 C CNN
+F 2 "Connector_PinHeader_2.54mm:PinHeader_1x03_P2.54mm_Vertical" H 2800 2650 50  0001 C CNN
 F 3 "~" H 2800 2650 50  0001 C CNN
 	1    2800 2650
@@
 F 0 "J2" H 2908 3331 50  0000 C CNN
 F 1 "Conn_01x01_Male" H 2908 3240 50  0000 C CNN
-F 2 "" H 2800 3150 50  0001 C CNN
+F 2 "Connector_PinHeader_2.54mm:PinHeader_1x01_P2.54mm_Vertical" H 2800 3150 50  0001 C CNN
 F 3 "~" H 2800 3150 50  0001 C CNN
 	1    2800 3150
@@
 F 0 "J3" H 2908 3731 50  0000 C CNN
 F 1 "Conn_01x02_Male" H 2908 3640 50  0000 C CNN
-F 2 "" H 2800 3550 50  0001 C CNN
+F 2 "Connector_PinHeader_2.54mm:PinHeader_1x02_P2.54mm_Vertical" H 2800 3550 50  0001 C CNN
 F 3 "~" H 2800 3550 50  0001 C CNN
 	1    2800 3550
@@
 F 0 "J4" H 2908 4331 50  0000 C CNN
 F 1 "Conn_01x02_Male" H 2908 4240 50  0000 C CNN
-F 2 "" H 2800 4150 50  0001 C CNN
+F 2 "Connector_PinHeader_2.54mm:PinHeader_1x02_P2.54mm_Vertical" H 2800 4150 50  0001 C CNN
 F 3 "~" H 2800 4150 50  0001 C CNN
 	1    2800 4150
@@
 F 0 "R1" H 6018 2946 50  0000 L CNN
 F 1 "10k" H 6018 2855 50  0000 L CNN
-F 2 "" V 5990 2890 50  0001 C CNN
+F 2 "Resistor_THT:R_Axial_DIN0207_L6.3mm_D2.5mm_P7.62mm_Horizontal" V 5990 2890 50  0001 C CNN
 F 3 "~" H 5950 2900 50  0001 C CNN
 	1    5950 2900
@@
 F 0 "R2" H 6018 3346 50  0000 L CNN
 F 1 "10k" H 6018 3255 50  0000 L CNN
-F 2 "" V 5990 3290 50  0001 C CNN
+F 2 "Resistor_THT:R_Axial_DIN0207_L6.3mm_D2.5mm_P7.62mm_Horizontal" V 5990 3290 50  0001 C CNN
 F 3 "~" H 5950 3300 50  0001 C CNN
 	1    5950 3300
@@
 F 0 "R3" H 6018 3746 50  0000 L CNN
 F 1 "10k" H 6018 3655 50  0000 L CNN
-F 2 "" V 5990 3690 50  0001 C CNN
+F 2 "Resistor_THT:R_Axial_DIN0207_L6.3mm_D2.5mm_P7.62mm_Horizontal" V 5990 3690 50  0001 C CNN
 F 3 "~" H 5950 3700 50  0001 C CNN
 	1    5950 3700

Commit message: finish adding footprints, including custom one for 1/4" mono jack; do rough part layout
Parts:
- J6: footprint (none) -> piano-keyboard-end-pcb:Switchcraft_RA49B11
- RV1, RV2: footprint (none) -> Potentiometer_THT:Potentiometer_Bourns_PTV09A-2_Single_Horizontal
- SW1, SW2, SW3, SW4, SW5, SW6, SW7: footprint (none) -> Button_Switch_THT:SW_PUSH_6mm
Changed lines of the file:
@@
 F 0 "RV1" H 3833 1396 50  0000 R CNN
 F 1 "R_POT_US" H 3833 1305 50  0000 R CNN
-F 2 "" H 3900 1350 50  0001 C CNN
+F 2 "Potentiometer_THT:Potentiometer_Bourns_PTV09A-2_Single_Horizontal" H 3900 1350 50  0001 C CNN
 F 3 "~" H 3900 1350 50  0001 C CNN
 	1    3900 1350
@@
 F 0 "RV2" H 4483 1396 50  0000 R CNN
 F 1 "R_POT_US" H 4483 1305 50  0000 R CNN
-F 2 "" H 4550 1350 50  0001 C CNN
+F 2 "Potentiometer_THT:Potentiometer_Bourns_PTV09A-2_Single_Horizontal" H 4550 1350 50  0001 C CNN
 F 3 "~" H 4550 1350 50  0001 C CNN
 	1    4550 1350
@@
 F 0 "J6" H 10982 1275 50  0000 C CNN
 F 1 "AudioJack2" H 10982 1184 50  0000 C CNN
-F 2 "" H 10950 950 50  0001 C CNN
+F 2 "piano-keyboard-end-pcb:Switchcraft_RA49B11" H 10950 950 50  0001 C CNN
 F 3 "~" H 10950 950 50  0001 C CNN
 	1    10950 950
@@
 F 0 "SW7" V 7704 998 50  0000 L CNN
 F 1 "SW_Push" V 7795 998 50  0000 L CNN
-F 2 "" H 7750 1050 50  0001 C CNN
+F 2 "Button_Switch_THT:SW_PUSH_6mm" H 7750 1050 50  0001 C CNN
 F 3 "~" H 7750 1050 50  0001 C CNN
 	1    7750 850
@@
 F 0 "SW6" V 8104 1348 50  0000 L CNN
 F 1 "SW_Push" V 8195 1348 50  0000 L CNN
-F 2 "" H 8150 1400 50  0001 C CNN
+F 2 "Button_Switch_THT:SW_PUSH_6mm" H 8150 1400 50  0001 C CNN
 F 3 "~" H 8150 1400 50  0001 C CNN
 	1    8150 1200
@@
 F 0 "SW5" V 8604 998 50  0000 L CNN
 F 1 "SW_Push" V 8695 998 50  0000 L CNN
-F 2 "" H 8650 1050 50  0001 C CNN
+F 2 "Button_Switch_THT:SW_PUSH_6mm" H 8650 1050 50  0001 C CNN
 F 3 "~" H 8650 1050 50  0001 C CNN
 	1    8650 850
@@
 F 0 "SW4" V 9004 1348 50  0000 L CNN
 F 1 "SW_Push" V 9095 1348 50  0000 L CNN
-F 2 "" H 9050 1400 50  0001 C CNN
+F 2 "Button_Switch_THT:SW_PUSH_6mm" H 9050 1400 50  0001 C CNN
 F 3 "~" H 9050 1400 50  0001 C CNN
 	1    9050 1200
@@
 F 0 "SW3" V 9404 998 50  0000 L CNN
 F 1 "SW_Push" V 9495 998 50  0000 L CNN
-F 2 "" H 9450 1050 50  0001 C CNN
+F 2 "Button_Switch_THT:SW_PUSH_6mm" H 9450 1050 50  0001 C CNN
 F 3 "~" H 9450 1050 50  0001 C CNN
 	1    9450 850
@@
 F 0 "SW2" V 9804 1348 50  0000 L CNN
 F 1 "SW_Push" V 9895 1348 50  0000 L CNN
-F 2 "" H 9850 1400 50  0001 C CNN
+F 2 "Button_Switch_THT:SW_PUSH_6mm" H 9850 1400 50  0001 C CNN
 F 3 "~" H 9850 1400 50  0001 C CNN
 	1    9850 1200
@@
 F 0 "SW1" V 10104 998 50  0000 L CNN
 F 1 "SW_Push" V 10195 998 50  0000 L CNN
-F 2 "" H 10150 1050 50  0001 C CNN
+F 2 "Button_Switch_THT:SW_PUSH_6mm" H 10150 1050 50  0001 C CNN
 F 3 "~" H 10150 1050 50  0001 C CNN
 	1    10150 850
