File: end-pcb/piano-keyboard-end-pcb.sch (KiCad schematic (older format))
At the start: 21 parts, among them J1 Conn_01x03_Male, J2 Conn_01x01_Male, J3 Conn_01x02_Male, J4 Conn_01x02_Male, J5 Conn_01x05_Female, J6 AudioJack2, SW1 SW_Push, SW2 SW_Push, SW3 SW_Push, SW4 SW_Push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

Commit message: make end PCB use Teensy pin 9 instead of MOSI, to match the software
Also move the Teensy down to make room for the new connection, and
reroute traces and rearrange silkscreen to compensate. Also add the
github URL where this repo will be to the silkscreen.
Parts:
- removed J4: Conn_01x02_Male, Connector_PinHeader_2.54mm:PinHeader_1x02_P2.54mm_Vertical, symbol Connector:Conn_01x02_Male
- added J4, J5: Conn_01x01_Male, Connector_PinHeader_2.54mm:PinHeader_1x01_P2.54mm_Vertical, symbol Connector:Conn_01x01_Male
- renumbered J5 to J6, J6 to J7
Connections:
- net MISO-DATA_OUT: now also J4.1 (Pin_1)
- net MOSI-SHIFT renamed 9-SHIFT
- net 9-SHIFT: now also J5.1 (Pin_1)
Changed lines of the file:
@@
 $EndDescr
 $Comp
-L Connector:Conn_01x05_Female J5
+L Connector:Conn_01x05_Female J6
 U 1 1 5E5EDAC0
 P 10400 5200
-F 0 "J5" H 10428 5226 50  0000 L CNN
+F 0 "J6" H 10428 5226 50  0000 L CNN
 F 1 "Conn_01x05_Female" H 10428 5135 50  0000 L CNN
 F 2 "Connector_PinSocket_2.54mm:PinSocket_1x05_P2.54mm_Horizontal" H 10400 5200 50  0001 C CNN
@@
 Wire Wire Line
 	5500 2550 5500 5200
-$Comp
-L Connector:Conn_01x02_Male J4
-U 1 1 5EE0F82F
-P 2800 4150
-F 0 "J4" H 2908 4331 50  0000 C CNN
-F 1 "Conn_01x02_Male" H 2908 4240 50  0000 C CNN
-F 2 "Connector_PinHeader_2.54mm:PinHeader_1x02_P2.54mm_Vertical" H 2800 4150 50  0001 C CNN
-F 3 "~" H 2800 4150 50  0001 C CNN
-	1    2800 4150
-	1    0    0    -1
-$EndComp
 Text Label 3000 4150 0    50   ~ 0
 MISO-DATA_OUT
-Text Label 3000 4250 0    50   ~ 0
-MOSI-SHIFT
-Wire Wire Line
-	6400 4250 6400 5300
-Wire Wire Line
-	6400 5300 7300 5300
-Wire Wire Line
-	3000 4250 6400 4250
-$Comp
-L Connector:AudioJack2 J6
+Text Label 3000 4400 0    50   ~ 0
+9-SHIFT
+Wire Wire Line
+	5450 5300 7300 5300
+$Comp
+L Connector:AudioJack2 J7
 U 1 1 5EE1C0C0
 P 10950 950
-F 0 "J6" H 10982 1275 50  0000 C CNN
+F 0 "J7" H 10982 1275 50  0000 C CNN
 F 1 "AudioJack2" H 10982 1184 50  0000 C CNN
 F 2 "piano-keyboard-end-pcb:Switchcraft_RA49B11" H 10950 950 50  0001 C CNN
@@
 Text Label 3000 3150 0    50   ~ 0
 5V
+$Comp
+L Connector:Conn_01x01_Male J4
+U 1 1 5EE819A7
+P 2800 4150
+F 0 "J4" H 2908 4331 50  0000 C CNN
+F 1 "Conn_01x01_Male" H 2908 4240 50  0000 C CNN
+F 2 "Connector_PinHeader_2.54mm:PinHeader_1x01_P2.54mm_Vertical" H 2800 4150 50  0001 C CNN
+F 3 "~" H 2800 4150 50  0001 C CNN
+	1    2800 4150
+	1    0    0    -1
+$EndComp
+$Comp
+L Connector:Conn_01x01_Male J5
+U 1 1 5EE8217E
+P 2800 4400
+F 0 "J5" H 2908 4581 50  0000 C CNN
+F 1 "Conn_01x01_Male" H 2908 4490 50  0000 C CNN
+F 2 "Connector_PinHeader_2.54mm:PinHeader_1x01_P2.54mm_Vertical" H 2800 4400 50  0001 C CNN
+F 3 "~" H 2800 4400 50  0001 C CNN
+	1    2800 4400
+	1    0    0    -1
+$EndComp
+Wire Wire Line
+	5450 4400 5450 5300
+Wire Wire Line
+	3000 4400 5450 4400
 $EndSCHEMATC

Commit message: use 3.3V throughout, instead of mixing it with 5V levels
This fixes the issues with the highest few keys intermittently not
working. It also makes the end PCB a little simpler. The shift registers
won't run as fast, but it turns out they don't need to.
Parts:
- removed J2: Conn_01x01_Male, Connector_PinHeader_2.54mm:PinHeader_1x01_P2.54mm_Vertical, symbol Connector:Conn_01x01_Male
- removed R1, R2, R3: 10k, Resistor_THT:R_Axial_DIN0207_L6.3mm_D2.5mm_P7.62mm_Horizontal, symbol Device:R_US
Connections:
- net +3V3 is gone; now on net VCC: J3.2 (Pin_2), RV1.1, RV2.1
- net MISO-DATA_OUT: now also U1.9 (QH)
Changed lines of the file:
@@
 Title "Modular Piano Keyboard End"
 Date "2020-06-06"
-Rev "v1"
+Rev "v2"
 Comp ""
 Comment1 ""
@@
 $EndComp
 $Comp
-L Connector:Conn_01x01_Male J2
-U 1 1 5EDDDC79
-P 2800 3150
-F 0 "J2" H 2908 3331 50  0000 C CNN
-F 1 "Conn_01x01_Male" H 2908 3240 50  0000 C CNN
-F 2 "Connector_PinHeader_2.54mm:PinHeader_1x01_P2.54mm_Vertical" H 2800 3150 50  0001 C CNN
-F 3 "~" H 2800 3150 50  0001 C CNN
-	1    2800 3150
-	1    0    0    -1
-$EndComp
-$Comp
 L Connector:Conn_01x02_Male J3
 U 1 1 5EDDE3D9
@@
 Text Label 3000 2750 0    50   ~ 0
 A1-MOD
-$Comp
-L power:VCC #PWR01
-U 1 1 5EDE6477
-P 3900 3150
-F 0 "#PWR01" H 3900 3000 50  0001 C CNN
-F 1 "VCC" H 3917 3323 50  0000 C CNN
-F 2 "" H 3900 3150 50  0001 C CNN
-F 3 "" H 3900 3150 50  0001 C CNN
-	1    3900 3150
-	1    0    0    -1
-$EndComp
-$Comp
-L power:PWR_FLAG #FLG01
-U 1 1 5EDE7A50
-P 3650 3150
-F 0 "#FLG01" H 3650 3225 50  0001 C CNN
-F 1 "PWR_FLAG" H 3650 3323 50  0000 C CNN
-F 2 "" H 3650 3150 50  0001 C CNN
-F 3 "~" H 3650 3150 50  0001 C CNN
-	1    3650 3150
-	1    0    0    -1
-$EndComp
-Connection ~ 3650 3150
-Wire Wire Line
-	3650 3150 3900 3150
 $Comp
 L power:PWR_FLAG #FLG02
@@
 	1    0    0    -1
 $EndComp
-$Comp
-L power:+3V3 #PWR02
-U 1 1 5EDEB14A
-P 3900 3700
-F 0 "#PWR02" H 3900 3550 50  0001 C CNN
-F 1 "+3V3" H 3915 3873 50  0000 C CNN
-F 2 "" H 3900 3700 50  0001 C CNN
-F 3 "" H 3900 3700 50  0001 C CNN
-	1    3900 3700
-	1    0    0    -1
-$EndComp
 Wire Wire Line
 	3800 3550 3800 3450
@@
 	1    0    0    -1
 $EndComp
-$Comp
-L power:+3V3 #PWR04
-U 1 1 5EDF56F3
-P 3900 1100
-F 0 "#PWR04" H 3900 950 50  0001 C CNN
-F 1 "+3V3" H 3915 1273 50  0000 C CNN
-F 2 "" H 3900 1100 50  0001 C CNN
-F 3 "" H 3900 1100 50  0001 C CNN
-	1    3900 1100
-	1    0    0    -1
-$EndComp
 Wire Wire Line
 	3900 1200 3900 1100
@@
 F 3 "" H 4550 1600 50  0001 C CNN
 	1    4550 1600
-	1    0    0    -1
-$EndComp
-$Comp
-L power:+3V3 #PWR06
-U 1 1 5EDFA2A9
-P 4550 1100
-F 0 "#PWR06" H 4550 950 50  0001 C CNN
-F 1 "+3V3" H 4565 1273 50  0000 C CNN
-F 2 "" H 4550 1100 50  0001 C CNN
-F 3 "" H 4550 1100 50  0001 C CNN
-	1    4550 1100
 	1    0    0    -1
 $EndComp
@@
 Wire Wire Line
 	6400 1850 6400 1950
-$Comp
-L Device:R_US R1
-U 1 1 5EE99843
-P 5950 2900
-F 0 "R1" H 6018 2946 50  0000 L CNN
-F 1 "10k" H 6018 2855 50  0000 L CNN
-F 2 "Resistor_THT:R_Axial_DIN0207_L6.3mm_D2.5mm_P7.62mm_Horizontal" V 5990 2890 50  0001 C CNN
-F 3 "~" H 5950 2900 50  0001 C CNN
-	1    5950 2900
-	1    0    0    -1
-$EndComp
-$Comp
-L Device:R_US R2
-U 1 1 5EE9C4B8
-P 5950 3300
-F 0 "R2" H 6018 3346 50  0000 L CNN
-F 1 "10k" H 6018 3255 50  0000 L CNN
-F 2 "Resistor_THT:R_Axial_DIN0207_L6.3mm_D2.5mm_P7.62mm_Horizontal" V 5990 3290 50  0001 C CNN
-F 3 "~" H 5950 3300 50  0001 C CNN
-	1    5950 3300
-	1    0    0    -1
-$EndComp
-$Comp
-L Device:R_US R3
-U 1 1 5EE9E9C9
-P 5950 3700
-F 0 "R3" H 6018 3746 50  0000 L CNN
-F 1 "10k" H 6018 3655 50  0000 L CNN
-F 2 "Resistor_THT:R_Axial_DIN0207_L6.3mm_D2.5mm_P7.62mm_Horizontal" V 5990 3690 50  0001 C CNN
-F 3 "~" H 5950 3700 50  0001 C CNN
-	1    5950 3700
-	1    0    0    -1
-$EndComp
-$Comp
-L power:GND #PWR08
-U 1 1 5EEA0F60
-P 5950 3900
-F 0 "#PWR08" H 5950 3650 50  0001 C CNN
-F 1 "GND" H 5955 3727 50  0000 C CNN
-F 2 "" H 5950 3900 50  0001 C CNN
-F 3 "" H 5950 3900 50  0001 C CNN
-	1    5950 3900
-	1    0    0    -1
-$EndComp
-Wire Wire Line
-	6200 2650 5950 2650
-Wire Wire Line
-	5950 2650 5950 2750
-Wire Wire Line
-	5950 3050 5950 3100
-Wire Wire Line
-	5950 3450 5950 3550
-Wire Wire Line
-	5700 4150 5700 3100
-Wire Wire Line
-	5700 3100 5950 3100
-Connection ~ 5950 3100
-Wire Wire Line
-	5950 3100 5950 3150
-Wire Wire Line
-	5950 3850 5950 3900
 Wire Wire Line
 	7950 5100 10200 5100
-Wire Wire Line
-	3000 3150 3650 3150
 Wire Wire Line
 	3000 3550 3650 3550
@@
 Text Label 3000 3650 0    50   ~ 0
 3.3V
-Text Label 3000 3150 0    50   ~ 0
-5V
 $Comp
 L Connector:Conn_01x01_Male J4
@@
 Wire Wire Line
 	3000 4400 5450 4400
+$Comp
+L power:VCC #PWR?
+U 1 1 5F132000
+P 3900 3700
+F 0 "#PWR?" H 3900 3550 50  0001 C CNN
+F 1 "VCC" H 3917 3873 50  0000 C CNN
+F 2 "" H 3900 3700 50  0001 C CNN
+F 3 "" H 3900 3700 50  0001 C CNN
+	1    3900 3700
+	1    0    0    -1
+$EndComp
+$Comp
+L power:VCC #PWR?
+U 1 1 5F137220
+P 3900 1100
+F 0 "#PWR?" H 3900 950 50  0001 C CNN
+F 1 "VCC" H 3917 1273 50  0000 C CNN
+F 2 "" H 3900 1100 50  0001 C CNN
+F 3 "" H 3900 1100 50  0001 C CNN
+	1    3900 1100
+	1    0    0    -1
+$EndComp
+$Comp
+L power:VCC #PWR?
+U 1 1 5F1375ED
+P 4550 1100
+F 0 "#PWR?" H 4550 950 50  0001 C CNN
+F 1 "VCC" H 4567 1273 50  0000 C CNN
+F 2 "" H 4550 1100 50  0001 C CNN
+F 3 "" H 4550 1100 50  0001 C CNN
+	1    4550 1100
+	1    0    0    -1
+$EndComp
+Wire Wire Line
+	5700 2650 6200 2650
+Wire Wire Line
+	5700 2650 5700 4150
 $EndSCHEMATC
